Commit message: IK scripts updated

File: Arm_Urdf/urdf/Arm_Urdf.urdf (robot description, URDF)
Before this commit: robot Arm_Urdf, 10 links, 9 joints
Joints:
- joint Joint_3: limit lower=0.00 upper=3.14 effort=50 velocity=5 -> lower=-1.00 upper=1.00 effort=50 velocity=5

Commit message: added new arm

File: Arm_Urdf/urdf/Arm_Urdf.urdf (robot description, URDF)
Before this commit: robot Arm_Urdf, 10 links, 9 joints
Links:
- added link camera_link, mass 1e-5; collision box size=0.025 0.025 0.025; visual box size=0.025 0.025 0.025
- added link camera_optical_link
Joints:
- added joint camera_joint: type fixed, parent Link_1, child camera_link, origin xyz=0.0 -0.02 0.02 rpy=0 0 -1.57, axis 0 1 0
- added joint camera_optical_joint: type fixed, parent camera_link, child camera_optical_link, origin xyz=0.0 0.0 0.0 rpy=-1.5707963 0 -1.5707963
